Commit message: 除了livox_laser_sim中的全局变量其余都更改完毕

File: livox_laser_simulation/urdf/livox_mid360.xacro (robot description, xacro)
@@ -52,5 +52,7 @@
 		  <samples>${samples}</samples>
 		  <downsample>${downsample}</downsample>
-		  <csv_file_name>/home/zjk/ranger_mid360_ur5_ws/src/livox_laser_simulation/scan_mode/mid360.csv</csv_file_name>
+      <!-- TAG:这里有全局变量 以解决-->
+		  <!-- <csv_file_name>/home/zjk/ranger_mid360_ur5_ws/src/livox_laser_simulation/scan_mode/mid360.csv</csv_file_name> -->
+		  <csv_file_name>$(find livox_laser_simulation)/scan_mode/mid360.csv</csv_file_name>
 		  <ros_topic>${ros_topic}</ros_topic>
         </plugin>
@@ -65,12 +67,21 @@
         <geometry>
           <!-- <mesh filename="/home/zjk/ranger_mid360_ur5_ws/src/livox_laser_simulation/meshes/mid360.dae"> -->
-          <mesh filename="/home/z/movebase3d_sim/src/livox_laser_simulation/meshes/mid360.dae">
+          <!-- TAG:这里的全局变量 已解决-->
+          <!-- <mesh filename="/home/z/movebase3d_sim/src/livox_laser_simulation/meshes/mid360.dae"> -->
+          <!-- </mesh> -->
+          <mesh filename="$(find livox_laser_simulation)/meshes/mid360.dae">
           </mesh>
         </geometry>
       </visual>
       <collision>
-		  <origin xyz="0 0 0" rpy="0 0 0" /> <geometry> <mesh
-		  filename="/home/z/movebase3d_sim/src/livox_laser_simulation/meshes/mid360_rules.dae">
-		  </mesh> </geometry>
+        <!-- TAG:这里的全局变量  已解决-->
+		  <origin xyz="0 0 0" rpy="0 0 0" /> <geometry>
+      <!-- <mesh  -->
+		  <!-- filename="/home/z/movebase3d_sim/src/livox_laser_simulation/meshes/mid360_rules.dae">  -->
+		  <!-- </mesh>  -->
+      <mesh
+		  filename="$(find livox_laser_simulation)/meshes/mid360_rules.dae">
+		  </mesh>
+      </geometry>
       </collision>
     </link>

File: livox_laser_simulation/urdf/mid360_IMU_platform.xacro (robot description, xacro)
@@ -38,5 +38,7 @@
       </joint>
       <!--lidar -->
-      <xacro:include filename="/home/zjk/ranger_mid360_ur5_ws/src/livox_laser_simulation/urdf/livox_mid360.xacro"/>
+      <!-- TAG:这里的全局变量 已经处理-->
+      <!-- <xacro:include filename="/home/zjk/ranger_mid360_ur5_ws/src/livox_laser_simulation/urdf/livox_mid360.xacro"/> -->
+      <xacro:include filename="$(find livox_laser_simulation)/urdf/livox_mid360.xacro"/>
       <!--xacro:Livox_Mid360 name="livox"/-->
     <!--imu -->

File: scout_simulator/scout_description/urdf/scout_v2.xacro (robot description, xacro)
@@ -44,5 +44,7 @@
     <!-- <xacro:include filename="/home/zjk/ranger_mid360_ur5_ws/src/livox_laser_simulation/urdf/livox_mid360.xacro"/> -->
     <!-- <xacro:include filename="/home/z/movebase3d_sim/src/livox_laser_simulation/urdf/livox_mid360.xacro"/> -->
-    <xacro:include filename="/home/z/movebase3d_scout_sim/src/livox_laser_simulation/urdf/livox_mid360.xacro"/>
+    <!-- TAG 这里有全局变量 已经处理 -->
+    <!-- <xacro:include filename="/home/z/movebase3d_scout_sim/src/livox_laser_simulation/urdf/livox_mid360.xacro"/> -->
+    <xacro:include filename="$(find livox_laser_simulation)/urdf/livox_mid360.xacro"/>
     <!--xacro:Livox_Mid360 name="livox"/-->
     <!--imu -->
